File: After Feedback/PCBs/Busra/EE463PCB_3.kicad_pcb (KiCad board)
At the start: 2 copper layers, 57 x 43.5 mm, 21 parts, among them J1 Conn_01x03, J2 Conn_01x02, Q1 IPD50R650CE, U1 HV9961LG-G

Commit message: PCB report updated.
Routing:
- net Net-(D7-Pad2): track 51.3 -> 43.3 mm, vias 0 -> 5
- net Net-(C1-Pad1): vias 2 -> 3
