File: After Feedback/PCBs/Busra/EE463PCB_3/EE463PCB_3.sch (KiCad schematic (older format))
At the start: 21 parts, among them J1 Conn_01x03, J2 Conn_01x02, Q1 IPD50R650CE, U1 HV9961LG-G

Commit message: Some files for presentation is uploaded
Connections:
- net at Q1.3 (S), R2.1, U1.2 (CS): now also C2.1, R3.1, U1.5 (PWMD), U1.6 (VDD), U1.7 (LD)
Other:
- moved on the sheet: C1, C2, C3, C4, C5, D1, D2, D3, D4, D5, D6, D7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
